Commit message: WIP:  wrench from effort

File: kortex_description/arms/gen3/6dof/urdf/gen3_macro.xacro (robot description, xacro)
@@ -31,4 +31,5 @@
     <!-- ros2 control include -->
     <xacro:include filename="$(find kortex_description)/arms/gen3/${dof}dof/urdf/kortex.ros2_control.xacro" />
+     <xacro:include filename="$(find kortex_description)/arms/gen3/${dof}dof/urdf/effort_force_torque_sensor.ros2_control.xacro"/>
     <xacro:kortex_ros2_control
       name="${prefix}KortexMultiInterfaceHardware" prefix="${prefix}"
@@ -372,3 +373,32 @@
     </xacro:if>
   </xacro:macro>
+   <!-- why the loading of this was being weird I don't know  -->
+  <!-- <xacro:macro name="effort_force_torque_sensor" params="name prefix use_mock_hardware:=^|true mock_sensor_commands:=^|false">
+    <!-- here was trying an external sensor before adding into the ros control xacro -->
+    <ros2_control name="${name}" type="sensor">
+      <hardware>
+          <plugin>kinova_effort_ft/EffortForceTorqueSensorHardware</plugin>
+          <param name="example_param_hw_start_duration_sec">0.0</param>
+          <param name="example_param_hw_stop_duration_sec">3.0</param>
+          <param name="example_param_max_sensor_change">5.0</param>
+      </hardware>
+      <sensor name="${prefix}tcp_fts_sensor">
+        <state_interface name="force.x"/>
+        <state_interface name="force.y"/>
+        <state_interface name="force.z"/>
+        <state_interface name="torque.x"/>
+        <state_interface name="torque.y"/>
+        <state_interface name="torque.z"/>
+        <param name="frame_id">end_effector_link</param>
+        <param name="fx_range">100</param>
+        <param name="fy_range">100</param>
+        <param name="fz_range">100</param>
+        <param name="tx_range">15</param>
+        <param name="ty_range">15</param>
+        <param name="tz_range">15</param>
+      </sensor>
+    </ros2_control>
+  </xacro:macro>
+  <xacro:external_rrbot_force_torque_sensor
+    name="ExternalRRBotFTSensor" prefix="$(arg prefix)"/> -->
 </robot>

File: kortex_description/arms/gen3/6dof/urdf/kortex.ros2_control.xacro (robot description, xacro)
@@ -128,4 +128,19 @@
         </joint>
       </xacro:if>
+      <sensor name="${prefix}tcp_fts_sensor">
+        <state_interface name="force.x"/>
+        <state_interface name="force.y"/>
+        <state_interface name="force.z"/>
+        <state_interface name="torque.x"/>
+        <state_interface name="torque.y"/>
+        <state_interface name="torque.z"/>
+        <param name="frame_id">end_effector_link</param>
+        <param name="fx_range">100</param>
+        <param name="fy_range">100</param>
+        <param name="fz_range">100</param>
+        <param name="tx_range">15</param>
+        <param name="ty_range">15</param>
+        <param name="tz_range">15</param>
+      </sensor>
     </ros2_control>
   </xacro:macro>

File: kortex_description/grippers/robotiq_2f_85/urdf/robotiq_2f_85_macro.xacro (robot description, xacro)
@@ -25,11 +25,6 @@
         include_ros2_control="${include_ros2_control}"
         com_port="${com_port}"
-        use_fake_hardware="${use_fake_hardware}"
-        mock_sensor_commands="${fake_sensor_commands}"
-        sim_gazebo="${sim_gazebo}"
-        sim_isaac="${sim_isaac}"
-        isaac_joint_commands="${isaac_joint_commands}"
-        isaac_joint_states="${isaac_joint_states}">
-        <origin xyz="0 0 0" rpy="0 0 0" />
+        use_fake_hardware="${use_fake_hardware}">
+                <origin xyz="0 0 0" rpy="0 0 0" />
     </xacro:robotiq_gripper>
   </xacro:macro>

Commit message: Merge of -> WIP:  wrench from effort

File: kortex_description/arms/gen3/6dof/urdf/gen3_macro.xacro (robot description, xacro)
@@ -33,4 +33,5 @@
     <!-- ros2 control include -->
     <xacro:include filename="$(find kortex_description)/arms/gen3/${dof}dof/urdf/kortex.ros2_control.xacro" />
+     <xacro:include filename="$(find kortex_description)/arms/gen3/${dof}dof/urdf/effort_force_torque_sensor.ros2_control.xacro"/>
     <xacro:kortex_ros2_control
       name="${prefix}KortexMultiInterfaceHardware" prefix="${prefix}"
@@ -375,3 +376,32 @@
     </xacro:if>
   </xacro:macro>
+   <!-- why the loading of this was being weird I don't know  -->
+  <!-- <xacro:macro name="effort_force_torque_sensor" params="name prefix use_mock_hardware:=^|true mock_sensor_commands:=^|false">
+    <!-- here was trying an external sensor before adding into the ros control xacro -->
+    <ros2_control name="${name}" type="sensor">
+      <hardware>
+          <plugin>kinova_effort_ft/EffortForceTorqueSensorHardware</plugin>
+          <param name="example_param_hw_start_duration_sec">0.0</param>
+          <param name="example_param_hw_stop_duration_sec">3.0</param>
+          <param name="example_param_max_sensor_change">5.0</param>
+      </hardware>
+      <sensor name="${prefix}tcp_fts_sensor">
+        <state_interface name="force.x"/>
+        <state_interface name="force.y"/>
+        <state_interface name="force.z"/>
+        <state_interface name="torque.x"/>
+        <state_interface name="torque.y"/>
+        <state_interface name="torque.z"/>
+        <param name="frame_id">end_effector_link</param>
+        <param name="fx_range">100</param>
+        <param name="fy_range">100</param>
+        <param name="fz_range">100</param>
+        <param name="tx_range">15</param>
+        <param name="ty_range">15</param>
+        <param name="tz_range">15</param>
+      </sensor>
+    </ros2_control>
+  </xacro:macro>
+  <xacro:external_rrbot_force_torque_sensor
+    name="ExternalRRBotFTSensor" prefix="$(arg prefix)"/> -->
 </robot>

File: kortex_description/arms/gen3/6dof/urdf/kortex.ros2_control.xacro (robot description, xacro)
@@ -132,4 +132,19 @@
         </joint>
       </xacro:if>
+      <sensor name="${prefix}tcp_fts_sensor">
+        <state_interface name="force.x"/>
+        <state_interface name="force.y"/>
+        <state_interface name="force.z"/>
+        <state_interface name="torque.x"/>
+        <state_interface name="torque.y"/>
+        <state_interface name="torque.z"/>
+        <param name="frame_id">end_effector_link</param>
+        <param name="fx_range">100</param>
+        <param name="fy_range">100</param>
+        <param name="fz_range">100</param>
+        <param name="tx_range">15</param>
+        <param name="ty_range">15</param>
+        <param name="tz_range">15</param>
+      </sensor>
     </ros2_control>
   </xacro:macro>

File: kortex_description/grippers/robotiq_2f_85/urdf/robotiq_2f_85_macro.xacro (robot description, xacro)
@@ -25,10 +25,10 @@
         include_ros2_control="${include_ros2_control}"
         com_port="${com_port}"
-        use_fake_hardware="${use_fake_hardware}"
-        fake_sensor_commands="${fake_sensor_commands}"
-        sim_ignition="${sim_ignition}"
-        sim_isaac="${sim_isaac}"
-        isaac_joint_commands="${isaac_joint_commands}"
-        isaac_joint_states="${isaac_joint_states}">
+        use_fake_hardware="${use_fake_hardware}">
+        <!-- fake_sensor_commands="${fake_sensor_commands}" -->
+        <!-- sim_ignition="${sim_ignition}" -->
+        <!-- sim_isaac="${sim_isaac}" -->
+        <!-- isaac_joint_commands="${isaac_joint_commands}" -->
+        <!-- isaac_joint_states="${isaac_joint_states}"> -->
         <origin xyz="0 0 0" rpy="0 0 0" />
     </xacro:robotiq_gripper>

Commit message: Seventh axis of destiny

File: kortex_description/arms/gen3/6dof/urdf/gen3_macro.xacro (robot description, xacro)
@@ -33,5 +33,4 @@
     <!-- ros2 control include -->
     <xacro:include filename="$(find kortex_description)/arms/gen3/${dof}dof/urdf/kortex.ros2_control.xacro" />
-     <xacro:include filename="$(find kortex_description)/arms/gen3/${dof}dof/urdf/effort_force_torque_sensor.ros2_control.xacro"/>
     <xacro:kortex_ros2_control
       name="${prefix}KortexMultiInterfaceHardware" prefix="${prefix}"
@@ -376,32 +375,3 @@
     </xacro:if>
   </xacro:macro>
-   <!-- why the loading of this was being weird I don't know  -->
-  <!-- <xacro:macro name="effort_force_torque_sensor" params="name prefix use_mock_hardware:=^|true mock_sensor_commands:=^|false">
-    <!-- here was trying an external sensor before adding into the ros control xacro -->
-    <ros2_control name="${name}" type="sensor">
-      <hardware>
-          <plugin>kinova_effort_ft/EffortForceTorqueSensorHardware</plugin>
-          <param name="example_param_hw_start_duration_sec">0.0</param>
-          <param name="example_param_hw_stop_duration_sec">3.0</param>
-          <param name="example_param_max_sensor_change">5.0</param>
-      </hardware>
-      <sensor name="${prefix}tcp_fts_sensor">
-        <state_interface name="force.x"/>
-        <state_interface name="force.y"/>
-        <state_interface name="force.z"/>
-        <state_interface name="torque.x"/>
-        <state_interface name="torque.y"/>
-        <state_interface name="torque.z"/>
-        <param name="frame_id">end_effector_link</param>
-        <param name="fx_range">100</param>
-        <param name="fy_range">100</param>
-        <param name="fz_range">100</param>
-        <param name="tx_range">15</param>
-        <param name="ty_range">15</param>
-        <param name="tz_range">15</param>
-      </sensor>
-    </ros2_control>
-  </xacro:macro>
-  <xacro:external_rrbot_force_torque_sensor
-    name="ExternalRRBotFTSensor" prefix="$(arg prefix)"/> -->
 </robot>

File: kortex_description/arms/gen3/7dof/urdf/kortex.ros2_control.xacro (robot description, xacro)
@@ -145,4 +145,19 @@
           </joint>
         </xacro:if>
+        <sensor name="${prefix}tcp_fts_sensor">
+          <state_interface name="force.x"/>
+          <state_interface name="force.y"/>
+          <state_interface name="force.z"/>
+          <state_interface name="torque.x"/>
+          <state_interface name="torque.y"/>
+          <state_interface name="torque.z"/>
+          <param name="frame_id">end_effector_link</param>
+          <param name="fx_range">100</param>
+          <param name="fy_range">100</param>
+          <param name="fz_range">100</param>
+          <param name="tx_range">15</param>
+          <param name="ty_range">15</param>
+          <param name="tz_range">15</param>
+        </sensor>
       </xacro:unless>
     </ros2_control>
