Commit message: Initial twist/moveit changes

File: kortex_description/arms/gen3/7dof/urdf/gen3_macro.xacro (robot description, xacro)
@@ -207,6 +207,6 @@
           xyz="0 0 1" />
         <limit
-          lower="${PI-0.01}"
-          upper="${PI+0.01}"
+          lower="${-2*PI}"
+          upper="${2*PI}"
           effort="39"
           velocity="1.3963" />

File: kortex_description/arms/gen3/7dof/urdf/kortex.ros2_control.xacro (robot description, xacro)
@@ -13,5 +13,5 @@
     use_internal_bus_gripper_comm:=true
     tf_prefix
-    initial_positions:=${dict(joint_1=0.0,joint_2=0.0,joint_3=0.0,joint_4=0.0,joint_5=0.0,joint_6=0.0,joint_7=0.0)}
+    initial_positions:=${dict(kinova_1=0.0,kinova_2=0.0,kinova_3=0.0,kinova_4=0.0,kinova_5=0.0,kinova_6=0.0,kinova_7=0.0)}
     robot_ip
     username
@@ -60,5 +60,5 @@
         </xacro:unless>
       </hardware>
-      <joint name="${prefix}joint_1">
+                <joint name="${prefix}joint_1">
         <command_interface name="position">
           <param name="min">{-2*pi}</param>
@@ -66,5 +66,6 @@
         </command_interface>
         <state_interface name="position">
-          <param name="initial_value">${initial_positions['joint_1']}</param>
+          <!-- <param name="initial_value">${initial_positions[prefix+'joint_1']}</param> -->
+          <param name="initial_value">0</param>
         </state_interface>
         <state_interface name="velocity"/>
@@ -77,5 +78,6 @@
         </command_interface>
         <state_interface name="position">
-          <param name="initial_value">${initial_positions['joint_2']}</param>
+          <!-- <param name="initial_value">${initial_positions[prefix+'joint_2']}</param> -->
+          <param name="initial_value">0</param>
         </state_interface>
         <state_interface name="velocity"/>
@@ -88,5 +90,6 @@
         </command_interface>
         <state_interface name="position">
-          <param name="initial_value">${initial_positions['joint_3']}</param>
+          <!-- <param name="initial_value">${initial_positions[prefix+'joint_3']}</param> -->
+          <param name="initial_value">0</param>
         </state_interface>
         <state_interface name="velocity"/>
@@ -99,5 +102,6 @@
         </command_interface>
         <state_interface name="position">
-          <param name="initial_value">${initial_positions['joint_4']}</param>
+          <!-- <param name="initial_value">${initial_positions[prefix+'joint_4']}</param> -->
+          <param name="initial_value">0</param>
         </state_interface>
         <state_interface name="velocity"/>
@@ -110,5 +114,6 @@
         </command_interface>
         <state_interface name="position">
-          <param name="initial_value">${initial_positions['joint_5']}</param>
+          <!-- <param name="initial_value">${initial_positions[prefix+'joint_5']}</param> -->
+          <param name="initial_value">0</param>
         </state_interface>
         <state_interface name="velocity"/>
@@ -121,5 +126,6 @@
         </command_interface>
         <state_interface name="position">
-          <param name="initial_value">${initial_positions['joint_6']}</param>
+          <!-- <param name="initial_value">${initial_positions[prefix+'joint_6']}</param> -->
+          <param name="initial_value">0</param>
         </state_interface>
         <state_interface name="velocity"/>
@@ -132,5 +138,6 @@
         </command_interface>
         <state_interface name="position">
-          <param name="initial_value">${initial_positions['joint_7']}</param>
+          <!-- <param name="initial_value">${initial_positions[prefix+'joint_7']}</param> -->
+          <param name="initial_value">0</param>
         </state_interface>
         <state_interface name="velocity"/>

Commit message: Use package for cad files for remote viewing ease

File: kortex_description/arms/gen3/7dof/urdf/gen3_macro.xacro (robot description, xacro)
@@ -70,14 +70,14 @@
         <origin xyz="0 0 0" rpy="0 0 0" />
         <geometry>
-          <mesh filename="file://$(find kortex_description)/arms/gen3/${dof}dof/meshes/base_link.dae" />
-        </geometry>
-        <material name="">
-          <color rgba="0.75294 0.75294 0.75294 1" />
-        </material>
-      </visual>
-      <collision>
-        <origin xyz="0 0 0" rpy="0 0 0" />
-        <geometry>
-          <mesh filename="file://$(find kortex_description)/arms/gen3/${dof}dof/meshes/base_link.dae" />
+          <mesh filename="package://kortex_description//arms/gen3/${dof}dof/meshes/base_link.dae" />
+        </geometry>
+        <material name="">
+          <color rgba="0.75294 0.75294 0.75294 1" />
+        </material>
+      </visual>
+      <collision>
+        <origin xyz="0 0 0" rpy="0 0 0" />
+        <geometry>
+          <mesh filename="package://kortex_description//arms/gen3/${dof}dof/meshes/base_link.dae" />
         </geometry>
       </collision>
@@ -92,14 +92,14 @@
         <origin xyz="0 0 0" rpy="0 0 0" />
         <geometry>
-          <mesh filename="file://$(find kortex_description)/arms/gen3/${dof}dof/meshes/shoulder_link.dae" />
-        </geometry>
-        <material name="">
-          <color rgba="0.75294 0.75294 0.75294 1" />
-        </material>
-      </visual>
-      <collision>
-        <origin xyz="0 0 0" rpy="0 0 0" />
-        <geometry>
-          <mesh filename="file://$(find kortex_description)/arms/gen3/${dof}dof/meshes/shoulder_link.dae" />
+          <mesh filename="package://kortex_description//arms/gen3/${dof}dof/meshes/shoulder_link.dae" />
+        </geometry>
+        <material name="">
+          <color rgba="0.75294 0.75294 0.75294 1" />
+        </material>
+      </visual>
+      <collision>
+        <origin xyz="0 0 0" rpy="0 0 0" />
+        <geometry>
+          <mesh filename="package://kortex_description//arms/gen3/${dof}dof/meshes/shoulder_link.dae" />
         </geometry>
       </collision>
@@ -148,14 +148,14 @@
         <origin xyz="0 0 0" rpy="0 0 0" />
         <geometry>
-          <mesh filename="file://$(find kortex_description)/arms/gen3/${dof}dof/meshes/half_arm_1_link.dae" />
-        </geometry>
-        <material name="">
-          <color rgba="0.75294 0.75294 0.75294 1" />
-        </material>
-      </visual>
-      <collision>
-        <origin xyz="0 0 0" rpy="0 0 0" />
-        <geometry>
-          <mesh filename="file://$(find kortex_description)/arms/gen3/${dof}dof/meshes/half_arm_1_link.dae" />
+          <mesh filename="package://kortex_description//arms/gen3/${dof}dof/meshes/half_arm_1_link.dae" />
+        </geometry>
+        <material name="">
+          <color rgba="0.75294 0.75294 0.75294 1" />
+        </material>
+      </visual>
+      <collision>
+        <origin xyz="0 0 0" rpy="0 0 0" />
+        <geometry>
+          <mesh filename="package://kortex_description//arms/gen3/${dof}dof/meshes/half_arm_1_link.dae" />
         </geometry>
       </collision>
@@ -182,14 +182,14 @@
         <origin xyz="0 0 0" rpy="0 0 0" />
         <geometry>
-          <mesh filename="file://$(find kortex_description)/arms/gen3/${dof}dof/meshes/half_arm_2_link.dae" />
-        </geometry>
-        <material name="">
-          <color rgba="0.75294 0.75294 0.75294 1" />
-        </material>
-      </visual>
-      <collision>
-        <origin xyz="0 0 0" rpy="0 0 0" />
-        <geometry>
-          <mesh filename="file://$(find kortex_description)/arms/gen3/${dof}dof/meshes/half_arm_2_link.dae" />
+          <mesh filename="package://kortex_description//arms/gen3/${dof}dof/meshes/half_arm_2_link.dae" />
+        </geometry>
+        <material name="">
+          <color rgba="0.75294 0.75294 0.75294 1" />
+        </material>
+      </visual>
+      <collision>
+        <origin xyz="0 0 0" rpy="0 0 0" />
+        <geometry>
+          <mesh filename="package://kortex_description//arms/gen3/${dof}dof/meshes/half_arm_2_link.dae" />
         </geometry>
       </collision>
@@ -238,14 +238,14 @@
         <origin xyz="0 0 0" rpy="0 0 0" />
         <geometry>
-          <mesh filename="file://$(find kortex_description)/arms/gen3/${dof}dof/meshes/forearm_link.dae" />
-        </geometry>
-        <material name="">
-          <color rgba="0.75294 0.75294 0.75294 1" />
-        </material>
-      </visual>
-      <collision>
-        <origin xyz="0 0 0" rpy="0 0 0" />
-        <geometry>
-          <mesh filename="file://$(find kortex_description)/arms/gen3/${dof}dof/meshes/forearm_link.dae" />
+          <mesh filename="package://kortex_description//arms/gen3/${dof}dof/meshes/forearm_link.dae" />
+        </geometry>
+        <material name="">
+          <color rgba="0.75294 0.75294 0.75294 1" />
+        </material>
+      </visual>
+      <collision>
+        <origin xyz="0 0 0" rpy="0 0 0" />
+        <geometry>
+          <mesh filename="package://kortex_description//arms/gen3/${dof}dof/meshes/forearm_link.dae" />
         </geometry>
       </collision>
@@ -272,14 +272,14 @@
         <origin xyz="0 0 0" rpy="0 0 0" />
         <geometry>
-          <mesh filename="file://$(find kortex_description)/arms/gen3/${dof}dof/meshes/spherical_wrist_1_link.dae" />
-        </geometry>
-        <material name="">
-          <color rgba="0.75294 0.75294 0.75294 1" />
-        </material>
-      </visual>
-      <collision>
-        <origin xyz="0 0 0" rpy="0 0 0" />
-        <geometry>
-          <mesh filename="file://$(find kortex_description)/arms/gen3/${dof}dof/meshes/spherical_wrist_1_link.dae" />
+          <mesh filename="package://kortex_description//arms/gen3/${dof}dof/meshes/spherical_wrist_1_link.dae" />
+        </geometry>
+        <material name="">
+          <color rgba="0.75294 0.75294 0.75294 1" />
+        </material>
+      </visual>
+      <collision>
+        <origin xyz="0 0 0" rpy="0 0 0" />
+        <geometry>
+          <mesh filename="package://kortex_description//arms/gen3/${dof}dof/meshes/spherical_wrist_1_link.dae" />
         </geometry>
       </collision>
@@ -328,14 +328,14 @@
         <origin xyz="0 0 0" rpy="0 0 0" />
         <geometry>
-          <mesh filename="file://$(find kortex_description)/arms/gen3/${dof}dof/meshes/spherical_wrist_2_link.dae" />
-        </geometry>
-        <material name="">
-          <color rgba="0.75294 0.75294 0.75294 1" />
-        </material>
-      </visual>
-      <collision>
-        <origin xyz="0 0 0" rpy="0 0 0" />
-        <geometry>
-          <mesh filename="file://$(find kortex_description)/arms/gen3/${dof}dof/meshes/spherical_wrist_2_link.dae" />
+          <mesh filename="package://kortex_description//arms/gen3/${dof}dof/meshes/spherical_wrist_2_link.dae" />
+        </geometry>
+        <material name="">
+          <color rgba="0.75294 0.75294 0.75294 1" />
+        </material>
+      </visual>
+      <collision>
+        <origin xyz="0 0 0" rpy="0 0 0" />
+        <geometry>
+          <mesh filename="package://kortex_description//arms/gen3/${dof}dof/meshes/spherical_wrist_2_link.dae" />
         </geometry>
       </collision>
@@ -363,14 +363,14 @@
         <origin xyz="0 0 0" rpy="0 0 0" />
         <geometry>
-          <mesh filename="file://$(find kortex_description)/arms/gen3/${dof}dof/meshes/bracelet_with_vision_link.dae" />
-        </geometry>
-        <material name="">
-          <color rgba="0.75294 0.75294 0.75294 1" />
-        </material>
-      </visual>
-      <collision>
-        <origin xyz="0 0 0" rpy="0 0 0" />
-        <geometry>
-          <mesh filename="file://$(find kortex_description)/arms/gen3/${dof}dof/meshes/bracelet_with_vision_link.dae" />
+          <mesh filename="package://kortex_description//arms/gen3/${dof}dof/meshes/bracelet_with_vision_link.dae" />
+        </geometry>
+        <material name="">
+          <color rgba="0.75294 0.75294 0.75294 1" />
+        </material>
+      </visual>
+      <collision>
+        <origin xyz="0 0 0" rpy="0 0 0" />
+        <geometry>
+          <mesh filename="package://kortex_description//arms/gen3/${dof}dof/meshes/bracelet_with_vision_link.dae" />
         </geometry>
       </collision>
@@ -387,14 +387,14 @@
         <origin xyz="0 0 0" rpy="0 0 0" />
         <geometry>
-          <mesh filename="file://$(find kortex_description)/arms/gen3/${dof}dof/meshes/bracelet_no_vision_link.dae" />
-        </geometry>
-        <material name="">
-          <color rgba="0.75294 0.75294 0.75294 1" />
-        </material>
-      </visual>
-      <collision>
-        <origin xyz="0 0 0" rpy="0 0 0" />
-        <geometry>
-          <mesh filename="file://$(find kortex_description)/arms/gen3/${dof}dof/meshes/bracelet_no_vision_link.dae" />
+          <mesh filename="package://kortex_description//arms/gen3/${dof}dof/meshes/bracelet_no_vision_link.dae" />
+        </geometry>
+        <material name="">
+          <color rgba="0.75294 0.75294 0.75294 1" />
+        </material>
+      </visual>
+      <collision>
+        <origin xyz="0 0 0" rpy="0 0 0" />
+        <geometry>
+          <mesh filename="package://kortex_description//arms/gen3/${dof}dof/meshes/bracelet_no_vision_link.dae" />
         </geometry>
       </collision>
